File: macintosh-portable-v1m.sch (KiCad schematic (older format))
At the start: 22 parts

Commit message: Finished V1M, more references on other sheets.
Parts:
- added CC5: C, symbol Device:C
- added RC1: ?, symbol Device:R_US
- added RC10: 7.6M, symbol Device:R_US
- added RC11: 4.65k, symbol Device:R_US
- added RC12: 7.5M, symbol Device:R_US
- added RC13, RC16, RC17: 99k, symbol Device:R_US
- added RC15: 265k, symbol Device:R_US
- added RC18: 386k, symbol Device:R_US
- added RC19, RC20: 98k, symbol Device:R_US
- added RC2: 1.37k, symbol Device:R_US
- added RC21, RC5: 100k, symbol Device:R_US
- added RC22: 19k, symbol Device:R_US
- added RC3: 97k, symbol Device:R_US
- added RC4: 78.5k, symbol Device:R_US
- added RC6: 960k, symbol Device:R_US
- added RC7: 320k, symbol Device:R_US
- added RC8: 360k, symbol Device:R_US
- added RC9: 9.7M, symbol Device:R_US
- CC7: renamed from CC?; value 4.7uF -> C
- RC14: renamed from RC1; value 3.8k -> 4.2k
- gave numbers to parts that had none: 1
- renumbered CC2 to CC1, CC1 to CC2, CC5 to CC6, CC6 to CC8
Connections:
- net GND: now also CC8.1, RC4.2, RC5.2, RC9.2; no longer CC8.2, OP1.2 (-)
- net V1M-17: now also RC11.2, RC12.1, RC17.2
- net V1M-19: now also RC13.2
- net V1M-22: now also RC17.1
- net V1M-25: now also RC15.2, RC16.1, RC20.2, RC6.2, RC8.2
- net V1M-33: now also RC21.2
- net V1M-37: now also QC3.3 (S)
- net V1M-38: now also RC18.2, RC19.2; no longer QC3.3 (S)
- net V1M-4: now also RC2.2, RC4.1
- net V1M-41: now also RC16.2
- net V1M-51: now also RC14.1, CC5.1, RC3.1; no longer RC14.2
- net V1M-52: now also RC10.2, RC2.1, RC8.1
- net V1M-62: now also RC1.2
- net V1M-8: now also RC6.1
- net at OP3.2 (-): now also RC14.2, CC5.2, RC15.1; no longer RC14.1
- net at OP3.3 (+), QC5.2 (D): now also RC18.1, RC19.1
- net at OP2.3 (+): now also RC5.1, RC7.1
- net at CC4.1, UC1.14 (B1+): now also RC11.1, RC9.1
- net at CC6.1, UC1.16 (OSC): now also RC12.2
- net at QC6.2 (D), QC7.1 (G): now also RC20.1
- net at QC7.2 (D), UC2.8 (V+): now also CC8.2; no longer CC8.1
- net at CC7.1, UC2.1 (FB/SHDN): now also RC21.1, RC22.1
- net at UC2.6 (VREF): now also RC22.2
- net at DC2.2 (A): now also RC10.1
- new net: OP1.2 (-), RC1.1, RC3.2
- new net V1M-11: RC13.1, RC7.2
- no-connect marks 11 -> 10
Other:
- note added: "Q1 drain\nenabled power charger\n(after resistors)"
- note added: "Q1 drain\nenabled power charger\nor battery available"
- note added: "Q1 gate\nenable power charger"
- note added: "Q1 source\npower charger"
- note added: "Q16 drain\nenabled RAM/TTL and\n2nd stage MOSFETs"
- note added: "Q16 gate\nenable RAM, TTL and \n2nd stage MOSFETs"
- note added: "To PMGR-33"
- note added: "enable +12V\n& SCSI cur."
- note added: "not connected"
- note added: "same as V1M-11"
- note added: "to PMGR-52\n(through resistor)"
- note added: "to SCSI power\nenable logic"
- moved on the sheet: CC1, CC2, CC3, CC4, CC6, CC7, CC8, DC1, DC2, OP2, QC1, QC2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

Commit message: Symbol library cleanup
Parts:
- DC1: symbol Reference_Voltage:LM385D-1.2 -> macintosh-portable:LM385D
- OP1, OP2, OP3: symbol Amplifier_Operational:OP20 -> macintosh-portable:OP20
- QC1, QC2, QC3, QC4, QC5, QC6, QC7: symbol Transistor_FET:IRF9020 -> macintosh-portable:IRF9020
- UC1: symbol Comparator:LTC1040CN -> macintosh-portable:LTC1040CN
Connections:
- wire segments 190 -> 192
Other:
- note added: "2x47uF capacitor\nto V1M-51"
- note added: "From\n74244 pin 3"
- note added: "From\nPMGR-31"
- note added: "From\nPMGR-38"
- note added: "Q1 & Q8\nEnable serial I/O ports"
- moved on the sheet: DC2, RC10, RC4
Changed lines of the file:
@@
 $Descr A4 11693 8268
 encoding utf-8
-Sheet 4 4
+Sheet 4 5
 Title "Macintosh Portable V1M Module"
 Date "2019-05-27"
@@
 $EndComp
 $Comp
-L Comparator:LTC1040CN UC1
+L macintosh-portable:LTC1040CN UC1
 U 3 1 5CEDE431
 P 6100 6850
@@
 	5600 7250 5700 7250
 $Comp
-L Transistor_FET:IRF9020 QC1
+L macintosh-portable:IRF9020 QC1
 U 1 1 5CEF3E9C
 P 4850 4900
@@
 V1M-40
 $Comp
-L Transistor_FET:IRF9020 QC5
+L macintosh-portable:IRF9020 QC5
 U 1 1 5CF00785
 P 3150 3650
@@
 Text HLabel 9750 5950 2    50   Input ~ 0
 V1M-31
-Text Notes 9750 5800 0    50   ~ 0
-100uF\nC16
 $Comp
 L Device:C CC7
@@
 V1M-37
 $Comp
-L Amplifier_Operational:OP20 OP1
+L macintosh-portable:OP20 OP1
 U 1 1 5CE65425
 P 6800 1100
@@
 V1M-51
 $Comp
-L Amplifier_Operational:OP20 OP2
+L macintosh-portable:OP20 OP2
 U 1 1 5CE5EDC3
 P 7300 2750
@@
 $EndComp
 $Comp
-L Amplifier_Operational:OP20 OP3
+L macintosh-portable:OP20 OP3
 U 1 1 5CE5AA98
 P 5500 3350
@@
 	2650 1550 5150 1550
 $Comp
-L Comparator:LTC1040CN UC1
+L macintosh-portable:LTC1040CN UC1
 U 1 1 5CE55934
 P 5550 1800
@@
 Wire Wire Line
 	5050 4900 9900 4900
-Text HLabel 1500 3650 0    50   Input ~ 0
-V1M-39
 Wire Wire Line
 	4750 4700 4750 4200
@@
 	-1   0    0    1
 $EndComp
-Connection ~ 2650 1000
 Wire Wire Line
 	2650 1000 1500 1000
@@
 $EndComp
 Wire Wire Line
-	2650 1000 6500 1000
-Wire Wire Line
 	6500 1200 6350 1200
 Wire Wire Line
@@
 Wire Wire Line
 	4500 3250 5200 3250
-Text HLabel 1500 650  0    50   Input ~ 0
-V1M-5
 $Comp
 L Device:R_US RC4
 U 1 1 5CEB0DD3
-P 2650 850
-F 0 "RC4" V 2445 850 50  0000 C CNN
-F 1 "78.5k" V 2536 850 50  0000 C CNN
-F 2 "" V 2690 840 50  0001 C CNN
-F 3 "~" H 2650 850 50  0001 C CNN
-	1    2650 850
+P 2650 750
+F 0 "RC4" V 2445 750 50  0000 C CNN
+F 1 "78.5k" V 2536 750 50  0000 C CNN
+F 2 "" V 2690 740 50  0001 C CNN
+F 3 "~" H 2650 750 50  0001 C CNN
+	1    2650 750
 	-1   0    0    1
 $EndComp
-Wire Wire Line
-	1500 650  2650 650
-Wire Wire Line
-	2650 650  2650 700
 $Comp
 L power:GND #PWR?
@@
 	6850 2850 7000 2850
 Wire Wire Line
-	5650 1250 5600 1250
-Wire Wire Line
-	5150 1250 5150 1550
+	5650 1300 5600 1300
+Wire Wire Line
+	5150 1300 5150 1550
 Connection ~ 5150 1550
 Wire Wire Line
 	5150 1550 5200 1550
 Wire Wire Line
-	5950 1250 6100 1250
-Wire Wire Line
-	6100 1250 6100 1800
+	5950 1300 6100 1300
+Wire Wire Line
+	6100 1300 6100 1800
 Connection ~ 6100 1800
 Wire Wire Line
@@
 L Device:R_US RC10
 U 1 1 5CF6A804
-P 5450 1250
-F 0 "RC10" V 5245 1250 50  0000 C CNN
-F 1 "7.6M" V 5336 1250 50  0000 C CNN
-F 2 "" V 5490 1240 50  0001 C CNN
-F 3 "~" H 5450 1250 50  0001 C CNN
-	1    5450 1250
+P 5450 1300
+F 0 "RC10" V 5245 1300 50  0000 C CNN
+F 1 "7.6M" V 5336 1300 50  0000 C CNN
+F 2 "" V 5490 1290 50  0001 C CNN
+F 3 "~" H 5450 1300 50  0001 C CNN
+	1    5450 1300
 	0    1    1    0
 $EndComp
 Wire Wire Line
-	5300 1250 5150 1250
+	5300 1300 5150 1300
 $Comp
 L Device:R_US RC20
@@
 $EndComp
 $Comp
-L Reference_Voltage:LM385D-1.2 DC1
+L macintosh-portable:LM385D DC1
 U 1 1 5CE6CF4E
 P 5900 2800
@@
 L Device:D DC2
 U 1 1 5D362828
-P 5800 1250
-F 0 "DC2" H 5750 1350 50  0000 L CNN
-F 1 "D" V 5845 1329 50  0001 L CNN
-F 2 "" H 5800 1250 50  0001 C CNN
-F 3 "~" H 5800 1250 50  0001 C CNN
-	1    5800 1250
+P 5800 1300
+F 0 "DC2" H 5750 1400 50  0000 L CNN
+F 1 "D" V 5845 1379 50  0001 L CNN
+F 2 "" H 5800 1300 50  0001 C CNN
+F 3 "~" H 5800 1300 50  0001 C CNN
+	1    5800 1300
 	-1   0    0    1
 $EndComp
@@
 	4050 2650 4500 2650
 $Comp
-L Comparator:LTC1040CN UC1
+L macintosh-portable:LTC1040CN UC1
 U 2 1 5CE7EB23
 P 4200 6250
@@
 	4750 6250 5400 6250
 $Comp
-L Transistor_FET:IRF9020 QC7
+L macintosh-portable:IRF9020 QC7
 U 1 1 5CF1AA8E
 P 4050 5250
@@
 	4750 3450 5200 3450
 $Comp
-L Transistor_FET:IRF9020 QC4
+L macintosh-portable:IRF9020 QC4
 U 1 1 5CF08979
 P 2200 3900
@@
 Wire Wire Line
 	1700 4000 1700 4200
-Text HLabel 2650 4950 2    50   Output ~ 0
+Text HLabel 2850 4950 2    50   Output ~ 0
 V1M-41
 Wire Wire Line
-	2650 4950 2200 4950
+	2850 4950 2200 4950
 Wire Wire Line
 	2200 4950 2200 5000
 $Comp
-L Transistor_FET:IRF9020 QC3
+L macintosh-portable:IRF9020 QC3
 U 1 1 5CF09852
 P 2100 4650
@@
 Wire Wire Line
 	1500 4650 1900 4650
-Wire Wire Line
-	1500 3650 2200 3650
-Wire Wire Line
-	2200 3700 2200 3650
-Connection ~ 2200 3650
-Wire Wire Line
-	2200 3650 2950 3650
 Text Notes 950  7150 0    50   ~ 0
 Q1 source\npower charger
 Text Notes 8850 4050 0    50   ~ 0
 Q1 gate\nenable power charger
-Text Notes 2600 4850 0    50   ~ 0
-enable +12V\n& SCSI cur.
 Text Notes 8900 2850 0    50   ~ 0
 Q16 gate\nenable RAM, TTL and \n2nd stage MOSFETs
@@
 	7700 1100 8500 1100
 Wire Wire Line
-	900  5700 900  3250
-Wire Wire Line
 	900  3250 3300 3250
 Connection ~ 4050 3250
@@
 	4750 3850 4750 4200
 $Comp
-L Transistor_FET:IRF9020 QC6
+L macintosh-portable:IRF9020 QC6
 U 1 1 5CF09F38
 P 3950 4450
@@
 V1M-21
 $Comp
-L Transistor_FET:IRF9020 QC2
+L macintosh-portable:IRF9020 QC2
 U 1 1 5CF0EE4C
 P 6350 4550
@@
 	0    1    1    0
 $EndComp
-Wire Wire Line
-	2200 5350 2200 5700
 Connection ~ 8000 2750
 Wire Wire Line
@@
 Wire Wire Line
 	3600 3250 4050 3250
-Wire Wire Line
-	900  5700 2200 5700
 Wire Wire Line
 	900  3250 900  2400
@@
 Text Notes 8900 2050 0    50   ~ 0
 not connected
+Text Notes 10200 5400 0    50   ~ 0
+Q1 & Q8\nEnable serial I/O ports
+Text Notes 10200 5800 0    50   ~ 0
+100uF\nC16
+Wire Wire Line
+	2200 5350 2200 5700
+Wire Wire Line
+	900  5700 900  3250
+Wire Wire Line
+	900  5700 2200 5700
+Wire Wire Line
+	2200 3650 2950 3650
+Connection ~ 2200 3650
+Wire Wire Line
+	2200 3700 2200 3650
+Wire Wire Line
+	1500 3650 2200 3650
+Text HLabel 1500 3650 0    50   Input ~ 0
+V1M-39
+Text Notes 2750 5200 0    50   ~ 0
+enable +12V\n& SCSI cur.
+Text Notes 1600 1350 0    50   ~ 0
+2x47uF capacitor\nto V1M-51
+$Comp
+L power:GND #PWR?
+U 1 1 5D06E311
+P 3050 650
+F 0 "#PWR?" H 3050 400 50  0001 C CNN
+F 1 "GND" H 3055 477 50  0000 C CNN
+F 2 "" H 3050 650 50  0001 C CNN
+F 3 "" H 3050 650 50  0001 C CNN
+	1    3050 650
+	1    0    0    -1
+$EndComp
+Connection ~ 2650 1000
+Wire Wire Line
+	2650 600  2650 550
+Wire Wire Line
+	2650 550  3050 550
+Wire Wire Line
+	3050 550  3050 650
+Wire Wire Line
+	2650 1000 6500 1000
+Wire Wire Line
+	2650 900  2650 1000
+Text Notes 850  950  0    50   ~ 0
+not connected
+Text Notes 650  4500 0    50   ~ 0
+From\nPMGR-38
+Text Notes 650  3700 0    50   ~ 0
+From\nPMGR-31
+Text Notes 550  4200 0    50   ~ 0
+not connected
+Text Notes 650  4750 0    50   ~ 0
+From\n74244 pin 3
 $EndSCHEMATC

Commit message: Progress on PMGR chip
Other:
- note added: "From PMGR-P1-3"
- note added: "From\n74244 O3b"
- note added: "From\nPMGR-P0-6"
- note added: "From\nPMGR-P1-5"
- note removed: "From\n74244 pin 3"
- note removed: "From\nPMGR-31"
- note removed: "From\nPMGR-38"
- note removed: "To PMGR-33"
Changed lines of the file:
@@
 $Descr A4 11693 8268
 encoding utf-8
-Sheet 4 5
+Sheet 3 5
 Title "Macintosh Portable V1M Module"
-Date "2019-05-27"
-Rev "0.12"
+Date "2019-06-08"
+Rev "0.13"
 Comp "https://oldcrap.org"
 Comment1 "Author: Pawel Pieczul"
@@
 Wire Wire Line
 	5950 5350 4250 5350
-Text HLabel 8450 4450 2    50   Output ~ 0
+Text HLabel 8450 4450 2    50   Input ~ 0
 V1M-19
 Wire Wire Line
@@
 not connected
 Text Notes 8850 4500 0    50   ~ 0
-To PMGR-33
+From PMGR-P1-3
 Text Notes 8900 3350 0    50   ~ 0
 Q16 drain\nenabled RAM/TTL and\n2nd stage MOSFETs
@@
 not connected
 Text Notes 650  4500 0    50   ~ 0
-From\nPMGR-38
-Text Notes 650  3700 0    50   ~ 0
-From\nPMGR-31
+From\nPMGR-P0-6
+Text Notes 600  3700 0    50   ~ 0
+From\nPMGR-P1-5
 Text Notes 550  4200 0    50   ~ 0
 not connected
 Text Notes 650  4750 0    50   ~ 0
-From\n74244 pin 3
+From\n74244 O3b
 $EndSCHEMATC

Commit message: Added reset circuit.
Other:
- note added: "to PMGR-IN-1\n(through resistor)"
- note removed: "to PMGR-52\n(through resistor)"
Changed lines of the file:
@@
 Title "Macintosh Portable V1M Module"
 Date "2019-06-08"
-Rev "0.13"
+Rev "0.14"
 Comp "https://oldcrap.org"
 Comment1 "Author: Pawel Pieczul"
@@
 same as V1M-11
 Text Notes 8900 1200 0    50   ~ 0
-to PMGR-52\n(through resistor)
+to PMGR-IN-1\n(through resistor)
 Text Notes 8900 2050 0    50   ~ 0
 not connected
